Commit message: Added D455 into the urdf model

File: urdf/electrical_excavator.urdf (robot description, URDF)
Before this commit: robot Machine, 6 links, 5 joints
Links:
- added link camera; visual mesh filename=package://autonomous_excavator/urdf/meshes/electrical/D455.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 scale=0.001 0.001 0.001
- added link camera_bracket; visual mesh filename=package://autonomous_excavator/urdf/meshes/electrical/Camer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 scale=0.001 0.001 0.001
Joints:
- added joint D455_fix: type fixed, parent camera_bracket, child camera, origin xyz=0.1065 0.0275 -0.0622 rpy=0 2.6180 0
- added joint camera_bracket_fix: type fixed, parent boom, child camera_bracket, origin xyz=0.3604 0.0495 0.1725 rpy=0 0 0

Commit message: Fixed the Arduino send and recive the actuators data in a non-sense order

File: urdf/electrical_excavator.urdf (robot description, URDF)
Before this commit: robot Machine, 8 links, 7 joints
Joints:
- joint Arm: origin xyz=1.050 0 0.210 rpy=0 0 0 -> xyz=1.071 0 0 rpy=0 0 0

Commit message: Fixed the location of the camera bracket

File: urdf/electrical_excavator.urdf (robot description, URDF)
Before this commit: robot Machine, 8 links, 7 joints
Joints:
- joint camera_bracket_fix: origin xyz=0.3604 0.0495 0.1725 rpy=0 0 0 -> xyz=0.3872 0.0495 0.0985 rpy=0 0.1974 0

Commit message: Implemented surface reconstruction display in Rviz2

File: urdf/electrical_excavator.urdf (robot description, URDF)
Before this commit: robot Machine, 8 links, 7 joints
Links:
- added link container
Joints:
- added joint container_fix: type fixed, parent world, child container, origin xyz=1.200 -0.013 -0.750 rpy=0 0 0

Commit message: Implemented marching cube visualization in Rviz2

File: urdf/electrical_excavator.urdf (robot description, URDF)
Before this commit: robot Machine, 9 links, 8 joints
Joints:
- joint container_fix: origin xyz=1.200 -0.013 -0.750 rpy=0 0 0 -> xyz=1.200 -0.130 -0.750 rpy=0 0 0

Commit message: Initial development commit

File: urdf/electrical_excavator.urdf (robot description, URDF)
Before this commit: robot Machine, 9 links, 8 joints
Joints:
- joint D455_fix: origin xyz=0.1065 0.0275 -0.0622 rpy=0 2.6180 0 -> xyz=0.1465 0.0275 -0.0622 rpy=0.09 2.6880 0
- joint container_fix: origin xyz=1.200 -0.130 -0.750 rpy=0 0 0 -> xyz=1.200 -0.430 -0.750 rpy=0 0 0
